File: REVISIONC.kicad_pcb (KiCad board)
At the start: 2 copper layers, 177.8 x 160 mm, 57 parts, among them J1 Conn_Coaxial, J10 Conn_02x03_Odd_Even, J2 Conn_Coaxial_Power, J3 Mini-DIN-6, J4 Conn_02x22_Odd_Even, J5 Conn_02x22_Odd_Even, J6 Conn_02x22_Odd_Even, J7 Conn_02x22_Odd_Even, J8 Conn_02x22_Odd_Even, J9 Conn_02x22_Odd_Even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

Commit message: Update REVISIONC.kicad_pcb
Other:
- board text added: "glibbi glorp"
- board text removed: "Max is awesome <3"
Changed lines of the file:
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@@
 		(layer "Edge.Cuts")
 	)
-	(gr_text "Max is awesome <3"
+	(gr_text "glibbi glorp"
 		(at 24.13 134.62 90)
 		(layer "F.Cu")
